File: ThumbsUp.kicad_pcb (KiCad board)
At the start: 2 copper layers, 123 parts, among them J1 Conn_01x18_Male, J10 Raiser_Male, J11 Raiser_Female, J12 Raiser_Male, J13 Raiser_Female, J14 Raiser_Male, J15 Raiser_Female, J16 Raiser_Male, J17 Raiser_Female, J18 Raiser_Male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

Commit message: Working on the layout
Parts:
- added J20: Conn_01x04_Female, Connector_PinSocket_2.54mm:PinSocket_1x04_P2.54mm_Vertical, F.Cu at (65.5, 328.5)
- added J21: Conn_01x04_Female, Connector_PinSocket_2.54mm:PinSocket_1x04_P2.54mm_Vertical, F.Cu at (113.1, 273.2)
- added J22: Conn_01x04_Female, Connector_PinSocket_2.54mm:PinSocket_1x04_P2.54mm_Vertical, F.Cu at (102.5, 301.8)
- added J23: Conn_01x04_Female, Connector_PinSocket_2.54mm:PinSocket_1x04_P2.54mm_Vertical, F.Cu at (102.5, 319.5)
- added J24: Conn_01x04_Male, Connector_PinHeader_2.54mm:PinHeader_1x04_P2.54mm_Vertical, F.Cu at (218.5, 331.0)
- added J25: Conn_01x04_Male, Connector_PinHeader_2.54mm:PinHeader_1x04_P2.54mm_Vertical, F.Cu at (170.5, 273.0)
- added J26: Conn_01x04_Male, Connector_PinHeader_2.54mm:PinHeader_1x04_P2.54mm_Vertical, F.Cu at (181.0, 308.5)
- added J27: Conn_01x04_Male, Connector_PinHeader_2.54mm:PinHeader_1x04_P2.54mm_Vertical, F.Cu at (181.0, 325.8)
- added J28: Conn_01x04_Female, Connector_PinSocket_2.54mm:PinSocket_1x04_P2.54mm_Vertical, F.Cu at (218.5, 331.0)
- added J29: Conn_01x04_Female, Connector_PinSocket_2.54mm:PinSocket_1x04_P2.54mm_Vertical, F.Cu at (170.5, 273.0)
- added J30: Conn_01x04_Female, Connector_PinSocket_2.54mm:PinSocket_1x04_P2.54mm_Vertical, F.Cu at (181.0, 308.5)
- added J31: Conn_01x04_Female, Connector_PinSocket_2.54mm:PinSocket_1x04_P2.54mm_Vertical, F.Cu at (181.0, 325.8)
- J1, J8: value Conn_01x18_Male -> Conn_01x04_Male; footprint Connector_PinHeader_2.54mm:PinHeader_1x18_P2.54mm_Vertical -> Connector_PinHeader_2.54mm:PinHeader_1x04_P2.54mm_Vertical
- J2, J7: value Conn_01x18_Female -> Conn_01x04_Male; footprint Connector_PinSocket_2.54mm:PinSocket_1x18_P2.54mm_Vertical -> Connector_PinHeader_2.54mm:PinHeader_1x04_P2.54mm_Vertical
- moved J5 235.2 mm to (183.8, 344.2), turned to 195 degrees
- moved J4 213.9 mm to (100.2, 342.8), turned to 165 degrees
- moved J1 195.6 mm to (65.5, 328.5)
- moved J3 189.1 mm to (100.2, 342.8), turned to 165 degrees
- moved J6 169.2 mm to (183.8, 344.2), turned to 195 degrees
- moved J7 162.7 mm to (102.5, 301.8), turned to 180 degrees
- moved J2 133.7 mm to (113.1, 273.2), turned to 270 degrees
- moved J8 132.3 mm to (102.5, 319.5), turned to 180 degrees
- moved MX30 14.0 mm to (155.8, 344.1), turned to 15 degrees
- moved MX18 11.7 mm to (127.7, 344.0), turned to 345 degrees
- moved MX26 9.88 mm to (173.7, 339.3), turned to 15 degrees
- moved MX31 8.49 mm to (191.0, 274.0)
- moved MX32 8.49 mm to (191.0, 291.5)
- moved MX33 8.49 mm to (191.0, 309.0)
- moved MX34 8.49 mm to (191.0, 326.5)
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Connections:
- J2 pad 1: COL0 -> Net-(J2-Pad1)
- J2 pad 2: COL1 -> Net-(J2-Pad2)
- J2 pad 3: COL2 -> Net-(J2-Pad3)
- J2 pad 4: COL3 -> Net-(J2-Pad4)
- J7 pad 1: COLB -> Net-(J7-Pad1)
- J7 pad 2: COLA -> Net-(J7-Pad2)
- J7 pad 3: COL9 -> Net-(J7-Pad3)
- J7 pad 4: COL8 -> Net-(J7-Pad4)
- MX1 pad 2: Net-(J1-Pad8) -> Net-(J2-Pad1)
- MX11 pad 2: Net-(J1-Pad5) -> Net-(J2-Pad4)
- MX12 pad 2: Net-(J1-Pad9) -> Net-(J7-Pad4)
- MX13 pad 1: Net-(J1-Pad4) -> Net-(J1-Pad1)
- MX13 pad 2: Net-(J1-Pad13) -> Net-(J8-Pad4)
- MX2 pad 2: Net-(J1-Pad12) -> Net-(J7-Pad1)
- MX3 pad 1: Net-(J1-Pad1) -> Net-(J1-Pad4)
- MX3 pad 2: Net-(J1-Pad16) -> Net-(J8-Pad1)
- MX31 pad 1: Net-(J8-Pad4) -> Net-(J28-Pad1)
- MX31 pad 2: Net-(J8-Pad5) -> Net-(J29-Pad4)
- MX32 pad 1: Net-(J8-Pad4) -> Net-(J28-Pad1)
- MX32 pad 2: Net-(J8-Pad9) -> Net-(J30-Pad4)
- MX33 pad 1: Net-(J8-Pad4) -> Net-(J28-Pad1)
- MX33 pad 2: Net-(J8-Pad13) -> Net-(J31-Pad4)
- MX35 pad 1: Net-(J8-Pad3) -> Net-(J28-Pad2)
- MX35 pad 2: Net-(J8-Pad6) -> Net-(J29-Pad3)
- MX36 pad 1: Net-(J8-Pad3) -> Net-(J28-Pad2)
- MX36 pad 2: Net-(J8-Pad10) -> Net-(J30-Pad3)
- MX37 pad 1: Net-(J8-Pad3) -> Net-(J28-Pad2)
- MX37 pad 2: Net-(J8-Pad14) -> Net-(J31-Pad3)
- MX39 pad 2: Net-(J8-Pad7) -> Net-(J29-Pad2)
- MX4 pad 2: Net-(J1-Pad7) -> Net-(J2-Pad2)
- MX40 pad 2: Net-(J8-Pad11) -> Net-(J30-Pad2)
- MX41 pad 1: Net-(J8-Pad2) -> Net-(J28-Pad3)
- MX41 pad 2: Net-(J8-Pad15) -> Net-(J31-Pad2)
- MX42 pad 2: Net-(J8-Pad8) -> Net-(J29-Pad1)
- MX43 pad 2: Net-(J8-Pad12) -> Net-(J30-Pad1)
- MX44 pad 1: Net-(J8-Pad1) -> Net-(J28-Pad4)
- MX44 pad 2: Net-(J8-Pad16) -> Net-(J31-Pad1)
- MX5 pad 2: Net-(J1-Pad11) -> Net-(J7-Pad2)
- MX6 pad 1: Net-(J1-Pad2) -> Net-(J1-Pad3)
- MX6 pad 2: Net-(J1-Pad15) -> Net-(J8-Pad2)
- MX7 pad 2: Net-(J1-Pad6) -> Net-(J2-Pad3)
- MX8 pad 2: Net-(J1-Pad10) -> Net-(J7-Pad3)
- MX9 pad 1: Net-(J1-Pad3) -> Net-(J1-Pad2)
- MX9 pad 2: Net-(J1-Pad14) -> Net-(J8-Pad3)

Commit message: Working on the layout
Parts:
- moved J14 253.5 mm to (136.8, 345.8), turned to 345 degrees
- moved J10 211.5 mm to (141.8, 284.8)
- moved J11 210.4 mm to (162.8, 350.0), turned to 105 degrees
- moved J9 203.4 mm to (141.8, 284.8)
- moved J16 203.1 mm to (113.0, 348.0), turned to 75 degrees
- moved J15 199.9 mm to (113.0, 348.0), turned to 75 degrees
- moved J12 186.5 mm to (162.8, 350.0), turned to 105 degrees
- moved J18 167.6 mm to (146.8, 345.8), turned to 15 degrees
- moved J17 165.0 mm to (146.8, 345.8), turned to 15 degrees
- moved J13 158.1 mm to (136.8, 345.8), turned to 345 degrees
Other:
- board outline added: 107 x 6.5 mm

Commit message: Working on the layout
Parts:
- moved J9 189.2 mm to (58.5, 114.8)
- moved J10 188.6 mm to (54.0, 117.8)
- moved C6 152.5 mm to (195.5, 59.0)
- moved C1 152.5 mm to (182.1, 72.5)
- moved C2 152.5 mm to (160.4, 93.7)
- moved C3 152.5 mm to (154.6, 98.3)
- moved C4 152.5 mm to (154.6, 101.2)
- moved C7 152.5 mm to (177.4, 78.8)
- moved C8 152.5 mm to (187.9, 65.8)
- moved C9 152.5 mm to (171.7, 81.5)
- moved D1 152.5 mm to (141.2, 110.8)
- moved D10 152.5 mm to (149.5, 101.8)
- moved D11 152.5 mm to (133.4, 117.5)
- moved D12 152.5 mm to (190.4, 61.5)
- moved D14 152.5 mm to (164.5, 90.5)
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Other:
- board size 107 x 6.5 mm -> 251.1 x 119.2 mm

Commit message: Split the boards
Parts:
- moved J13 260.9 mm to (118.9, 98.9)
- moved J5 260.9 mm to (215.1, 87.5)
- moved MX18 260.9 mm to (109.2, 93.3)
- moved MX22 260.9 mm to (94.4, 82.2)
- moved MX26 260.9 mm to (206.1, 82.1)
- moved MX30 260.9 mm to (191.4, 93.3)
- moved J17 260.9 mm to (181.3, 98.7)
- moved J3 260.9 mm to (85.4, 87.7)
- moved J23 137.8 mm to (106.8, 179.1)
- moved J22 137.6 mm to (113.7, 163.1)
- moved J11 137.4 mm to (191.7, 226.0)
- moved J14 137.4 mm to (115.4, 222.4)
- moved J15 137.4 mm to (95.7, 221.5)
- moved J21 137.4 mm to (120.2, 146.8)
- moved MX14 137.4 mm to (79.6, 187.4)
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Connections:
- J10 pad 1: Net-(J10-Pad1) -> (no net)
- J10 pad 2: Net-(J10-Pad2) -> (no net)
- J10 pad 3: Net-(J10-Pad3) -> (no net)
- J10 pad 4: Net-(J10-Pad4) -> (no net)
- J11 pad 1: Net-(J11-Pad1) -> (no net)
- J11 pad 2: Net-(J11-Pad2) -> (no net)
- J11 pad 3: Net-(J11-Pad3) -> (no net)
- J11 pad 4: Net-(J11-Pad4) -> (no net)
- J13 pad 1: Net-(J13-Pad1) -> (no net)
- J13 pad 2: Net-(J13-Pad2) -> (no net)
- J13 pad 3: Net-(J13-Pad3) -> (no net)
- J13 pad 4: Net-(J13-Pad4) -> (no net)
- J14 pad 1: Net-(J14-Pad1) -> (no net)
- J14 pad 2: Net-(J14-Pad2) -> (no net)
- J14 pad 3: Net-(J14-Pad3) -> (no net)
- J14 pad 4: Net-(J14-Pad4) -> (no net)
- J15 pad 1: Net-(J15-Pad1) -> (no net)
- J15 pad 2: Net-(J15-Pad2) -> (no net)
- J15 pad 3: Net-(J15-Pad3) -> (no net)
- J15 pad 4: Net-(J15-Pad4) -> (no net)
- J17 pad 1: VCC -> (no net)
- J17 pad 2: SDA -> (no net)
- J17 pad 3: SCL -> (no net)
- J17 pad 4: GND -> (no net)
- J18 pad 1: VCC -> (no net)
- J18 pad 2: SDA -> (no net)
- J18 pad 3: SCL -> (no net)
- J18 pad 4: GND -> (no net)
- J20 pad 1: COL3 -> (no net)
- J20 pad 2: COL2 -> (no net)
- J20 pad 3: COL1 -> (no net)
- J20 pad 4: COL0 -> (no net)
- J21 pad 1: Net-(D4-Pad2) -> (no net)
- J21 pad 2: Net-(D3-Pad2) -> (no net)
- J21 pad 3: Net-(D2-Pad2) -> (no net)
- J21 pad 4: Net-(D1-Pad2) -> (no net)
- J22 pad 1: Net-(D8-Pad2) -> (no net)
- J22 pad 2: Net-(D7-Pad2) -> (no net)
- J22 pad 3: Net-(D6-Pad2) -> (no net)
- J22 pad 4: Net-(D5-Pad2) -> (no net)
- J23 pad 1: Net-(D12-Pad2) -> (no net)
- J23 pad 2: Net-(D11-Pad2) -> (no net)
- J23 pad 3: Net-(D10-Pad2) -> (no net)
- J23 pad 4: Net-(D9-Pad2) -> (no net)
- J24 pad 1: COL8 -> (no net)
- J24 pad 2: COL9 -> (no net)
- J24 pad 3: COLA -> (no net)
- J24 pad 4: COLB -> (no net)
- J25 pad 1: Net-(D34-Pad2) -> (no net)
- J25 pad 2: Net-(D33-Pad2) -> (no net)
- J25 pad 3: Net-(D32-Pad2) -> (no net)
- J25 pad 4: Net-(D31-Pad2) -> (no net)
- J26 pad 1: Net-(D38-Pad2) -> (no net)
- J26 pad 2: Net-(D37-Pad2) -> (no net)
- J26 pad 3: Net-(D36-Pad2) -> (no net)
- J26 pad 4: Net-(D35-Pad2) -> (no net)
- J27 pad 1: Net-(D42-Pad2) -> (no net)
- J27 pad 2: Net-(D41-Pad2) -> (no net)
- J27 pad 3: Net-(D40-Pad2) -> (no net)
- J27 pad 4: Net-(D39-Pad2) -> (no net)
- J3 pad 1: Net-(J3-Pad1) -> (no net)
- J3 pad 2: Net-(J3-Pad2) -> (no net)
- J3 pad 3: Net-(J3-Pad3) -> (no net)
- J3 pad 4: Net-(J3-Pad4) -> (no net)
- J4 pad 1: COL4 -> (no net)
- J4 pad 2: Net-(D18-Pad2) -> (no net)
- J4 pad 3: Net-(D19-Pad2) -> (no net)
- J4 pad 4: COL5 -> (no net)
- J5 pad 1: Net-(J5-Pad1) -> (no net)
- J5 pad 2: Net-(J5-Pad2) -> (no net)
- J5 pad 3: Net-(J5-Pad3) -> (no net)
- J5 pad 4: Net-(J5-Pad4) -> (no net)
- J6 pad 1: COL6 -> (no net)
- J6 pad 2: Net-(D29-Pad2) -> (no net)
- J6 pad 3: Net-(D30-Pad2) -> (no net)
- J6 pad 4: COL7 -> (no net)
- J9 pad 1: Net-(J9-Pad1) -> (no net)
- J9 pad 2: Net-(J9-Pad2) -> (no net)
- J9 pad 3: Net-(J9-Pad3) -> (no net)
- J9 pad 4: Net-(J9-Pad4) -> (no net)
- MX10 pad 1: COL2 -> (no net)
- MX10 pad 2: Net-(D14-Pad2) -> (no net)
- MX14 pad 1: COL3 -> (no net)
- MX14 pad 2: Net-(D13-Pad2) -> (no net)
- MX15 pad 1: Net-(MX15-Pad1) -> (no net)
- MX15 pad 2: Net-(D15-Pad2) -> (no net)
- MX16 pad 1: Net-(MX16-Pad1) -> (no net)
- MX16 pad 2: Net-(D16-Pad2) -> (no net)
- MX17 pad 1: Net-(MX17-Pad1) -> (no net)
- MX17 pad 2: Net-(D17-Pad2) -> (no net)
- MX18 pad 1: Net-(J3-Pad1) -> (no net)
- MX18 pad 2: Net-(J3-Pad2) -> (no net)
- MX19 pad 1: Net-(MX19-Pad1) -> (no net)
- MX19 pad 2: Net-(D20-Pad2) -> (no net)
- MX20 pad 1: Net-(MX20-Pad1) -> (no net)
- MX20 pad 2: Net-(D21-Pad2) -> (no net)
- MX21 pad 1: Net-(MX21-Pad1) -> (no net)
- MX21 pad 2: Net-(D22-Pad2) -> (no net)
- MX22 pad 1: Net-(J3-Pad4) -> (no net)
- MX22 pad 2: Net-(J3-Pad3) -> (no net)
- MX23 pad 1: Net-(MX23-Pad1) -> (no net)
- MX23 pad 2: Net-(D23-Pad2) -> (no net)
- MX24 pad 1: Net-(MX24-Pad1) -> (no net)
- MX24 pad 2: Net-(D24-Pad2) -> (no net)
- MX25 pad 1: Net-(MX25-Pad1) -> (no net)
- MX25 pad 2: Net-(D25-Pad2) -> (no net)
- MX26 pad 1: Net-(J5-Pad1) -> (no net)
- MX26 pad 2: Net-(J5-Pad2) -> (no net)
- MX27 pad 1: Net-(MX27-Pad1) -> (no net)
- MX27 pad 2: Net-(D26-Pad2) -> (no net)
- MX28 pad 1: Net-(MX28-Pad1) -> (no net)
- MX28 pad 2: Net-(D27-Pad2) -> (no net)
- MX29 pad 1: Net-(MX29-Pad1) -> (no net)
- MX29 pad 2: Net-(D28-Pad2) -> (no net)
- MX30 pad 1: Net-(J5-Pad4) -> (no net)
- MX30 pad 2: Net-(J5-Pad3) -> (no net)
- MX34 pad 1: COL8 -> (no net)
- MX34 pad 2: Net-(D43-Pad2) -> (no net)
- MX38 pad 1: COL9 -> (no net)
- MX38 pad 2: Net-(D44-Pad2) -> (no net)
Other:
- board size 251.1 x 119.2 mm -> 251.1 x 336.1 mm
