File: ThumbsUp.kicad_pcb (KiCad board)
At the start: 2 copper layers, 251.1 x 336.1 mm, 143 parts, among them J1 Conn_01x04_Male, J10 Raiser_Male, J11 Raiser_Female, J12 Raiser_Male, J13 Raiser_Female, J14 Raiser_Male, J15 Raiser_Female, J16 Raiser_Male, J17 Raiser_Female, J18 Raiser_Male, J19 52559-1233, J2 Conn_01x04_Male, J20 Conn_01x04_Female, J21 Conn_01x04_Female, J22 Conn_01x04_Female, J23 Conn_01x04_Female, J24 Conn_01x04_Male, J25 Conn_01x04_Male, J26 Conn_01x04_Male, J27 Conn_01x04_Male, J28 Conn_01x04_Female, J29 Conn_01x04_Female, J3 Conn_01x04_Female, J30 Conn_01x04_Female, J31 Conn_01x04_Female, J4 Conn_01x04_Male, J5 Conn_01x04_Female, J6 Conn_01x04_Male, J7 Conn_01x04_Male, J8 Conn_01x04_Male, J9 Raiser_Female, SW1 SW_Push, U1 ATmega32U4-AU, Y1 16MHz

Commit message: Moved the touchpad connector
Parts:
- moved J19 40.9 mm to (173.5, 95.8), turned to 270 degrees
Routing:
- net SCL-TOP: track 61.4 -> 13.9 mm
- net VCC-TOP: track 59.5 -> 17.0 mm
- net SDA-TOP: track 59.8 -> 20.3 mm
- net GND-TOP: track 63.6 -> 41.7 mm

Commit message: Added pullup resistors for trackpad, re-produced the gerbers
Parts:
- removed the G*** at (146.1, 311.7)
- removed the G*** at (149.4, 62.5)
- removed the G*** at (144.3, 295.9)
- removed the G*** at (145.8, 174.2)
- removed the MX30 at (191.4, 93.3)
- added G***: LOGO, Silkscreens:Crowfeet75, B.Cu at (146.8, 314.9)
- added G***: LOGO, Silkscreens:Crowfeet75, F.Cu at (132.7, 209.8)
- added G***: LOGO, Silkscreens:Crowfeet75, F.Cu at (149.3, 54.6)
- added G***: LOGO, Silkscreens:Crowfeet75, F.Cu at (145.1, 314.6)
- added R5: 5.1K, Resistor_SMD:R_0805_2012Metric, B.Cu at (178.6, 95.5)
- added R6: 5.1K, Resistor_SMD:R_0805_2012Metric, B.Cu at (179.3, 102.7)
Routing:
- net SCL-TOP: track 13.9 -> 21.1 mm
- net VCC-TOP: track 17.0 -> 22.5 mm
- net SDA-TOP: track 20.3 -> 25.2 mm
