File: ThumbsUp.sch (KiCad schematic (older format))
At the start: 125 parts, among them J1 Conn_01x18_Male, J10 Raiser_Male, J11 Raiser_Female, J12 Raiser_Male, J13 Raiser_Female, J14 Raiser_Male, J15 Raiser_Female, J16 Raiser_Male, J17 Raiser_Female, J18 Raiser_Male, J2 Conn_01x18_Female, J3 Conn_01x04_Female, J4 Conn_01x04_Male, J5 Conn_01x04_Female, J6 Conn_01x04_Male, J7 Conn_01x18_Female, J8 Conn_01x18_Male, J9 Raiser_Female, SW1 SW_Push, U1 ATmega32U4-AU, Y1 16MHz

Commit message: Started the layout
Parts:
- added J19: 52559-1233, 525591233, symbol 52559-1233:52559-1233
- MX1, MX10, MX11, MX12, MX13, MX14, MX15, MX16, MX17, MX18, MX19, MX2, MX20, MX21, MX22, MX23, MX24, MX25, MX26, MX27, MX28, MX29, MX3, MX30, MX31, MX32, MX33, MX34, MX35, MX36, MX37, MX38, MX39, MX4, MX40, MX41, MX42, MX43, MX44, MX5, MX6, MX7, MX8, MX9: footprint SwitchFootprints:MX-Alps-Choc-KS32-X-1U-NoLED -> keyswitches:Kailh_socket_PG1350_optional
Connections:
- net GND: now also J17.4 (Pin_4), J18.4 (Pin_4), J19.11
- net VCC: now also J17.1 (Pin_1), J18.1 (Pin_1), J19.12
- net SCL: now reaches U1.18 (PD0)
- net SCL: now also J17.3 (Pin_3), J18.3 (Pin_3), J19.9
- net SDA: now reaches U1.19 (PD1)
- net SDA: now also J17.2 (Pin_2), J18.2 (Pin_2), J19.10
- no-connect marks 44 -> 36
Other:
- moved on the sheet: J17, J18

Commit message: Working on the layout
Parts:
- removed J1, J8: Conn_01x18_Male, Connector_PinHeader_2.54mm:PinHeader_1x18_P2.54mm_Vertical, symbol Connector:Conn_01x18_Male
- removed J2, J7: Conn_01x18_Female, Connector_PinSocket_2.54mm:PinSocket_1x18_P2.54mm_Vertical, symbol Connector:Conn_01x18_Female
- added J1, J2, J24, J25, J26, J27, J7, J8: Conn_01x04_Male, Connector_PinHeader_2.54mm:PinHeader_1x04_P2.54mm_Vertical, symbol Connector:Conn_01x04_Male
- added J20, J21, J22, J23, J28, J29, J30, J31: Conn_01x04_Female, Connector_PinSocket_2.54mm:PinSocket_1x04_P2.54mm_Vertical, symbol Connector:Conn_01x04_Female
Connections:
- net COL0: now also J20.4 (Pin_4)
- net COL1: now also J20.3 (Pin_3)
- net COL2: now also J20.2 (Pin_2)
- net COL3: now also J20.1 (Pin_1)
- net COL8: now also J24.1 (Pin_1)
- net COL9: now also J24.2 (Pin_2)
- net COLA: now also J24.3 (Pin_3)
- net COLB: now also J24.4 (Pin_4)
- net at MX1.2 (ROW): now also J2.1 (Pin_1)
- net at MX4.2 (ROW): now also J2.2 (Pin_2)
- net at MX2.2 (ROW): now also J7.1 (Pin_1)
- net at MX5.2 (ROW): now also J7.2 (Pin_2)
- net at MX7.2 (ROW): now also J2.3 (Pin_3)
- net at MX11.2 (ROW): now also J2.4 (Pin_4)
- net at MX8.2 (ROW): now also J7.3 (Pin_3)
- net at MX12.2 (ROW): now also J7.4 (Pin_4)
- net at MX3.1 (COL): now also J1.4 (Pin_4)
- net at MX3.2 (ROW): now also J8.1 (Pin_1)
- net at MX6.1 (COL): now also J1.3 (Pin_3)
- net at MX6.2 (ROW): now also J8.2 (Pin_2)
- net at MX9.1 (COL): now also J1.2 (Pin_2)
- net at MX9.2 (ROW): now also J8.3 (Pin_3)
- net at MX13.1 (COL): now also J1.1 (Pin_1)
- net at MX13.2 (ROW): now also J8.4 (Pin_4)
- net at D6.2 (A): now also J22.3 (Pin_3)
- net at D7.2 (A): now also J22.2 (Pin_2)
- net at D8.2 (A): now also J22.1 (Pin_1)
- net at D9.2 (A): now also J23.4 (Pin_4)
- net at D10.2 (A): now also J23.3 (Pin_3)
- net at D11.2 (A): now also J23.2 (Pin_2)
- net at D12.2 (A): now also J23.1 (Pin_1)
- net at D1.2 (A): now also J21.4 (Pin_4)
- net at D2.2 (A): now also J21.3 (Pin_3)
- net at D3.2 (A): now also J21.2 (Pin_2)
- net at D4.2 (A): now also J21.1 (Pin_1)
- net at D5.2 (A): now also J22.4 (Pin_4)
- net at MX42.2 (ROW): now also J29.1 (Pin_1)
- net at MX39.2 (ROW): now also J29.2 (Pin_2)
- net at MX43.2 (ROW): now also J30.1 (Pin_1)
- net at MX35.1 (COL), MX36.1 (COL), MX37.1 (COL): now also J28.2 (Pin_2)
- net at MX35.2 (ROW): now also J29.3 (Pin_3)
- net at MX31.1 (COL), MX32.1 (COL), MX33.1 (COL): now also J28.1 (Pin_1)
- net at MX31.2 (ROW): now also J29.4 (Pin_4)
- net at MX36.2 (ROW): now also J30.3 (Pin_3)
- net at MX32.2 (ROW): now also J30.4 (Pin_4)
- net at MX44.1 (COL): now also J28.4 (Pin_4)
- net at MX44.2 (ROW): now also J31.1 (Pin_1)
- net at MX41.1 (COL): now also J28.3 (Pin_3)
- net at MX41.2 (ROW): now also J31.2 (Pin_2)
- net at MX37.2 (ROW): now also J31.3 (Pin_3)
- net at MX33.2 (ROW): now also J31.4 (Pin_4)
- net at D36.2 (A): now also J26.3 (Pin_3)
- net at D37.2 (A): now also J26.2 (Pin_2)
- net at D38.2 (A): now also J26.1 (Pin_1)
- net at D39.2 (A): now also J27.4 (Pin_4)
- net at D40.2 (A): now also J27.3 (Pin_3)
- net at D41.2 (A): now also J27.2 (Pin_2)
- net at D42.2 (A): now also J27.1 (Pin_1)
- net at D31.2 (A): now also J25.4 (Pin_4)
- net at D32.2 (A): now also J25.3 (Pin_3)
- net at D33.2 (A): now also J25.2 (Pin_2)
- net at D34.2 (A): now also J25.1 (Pin_1)
- net at D35.2 (A): now also J26.4 (Pin_4)
- net at MX40.2 (ROW): now also J30.2 (Pin_2)
Changed lines of the file:
@@
 	1    0    0    -1
-$EndComp
-$Comp
-L Connector:Conn_01x18_Female J2
-U 1 1 620D7AD0
-P 5400 7600
-F 0 "J2" H 5300 8600 50  0000 C CNN
-F 1 "Conn_01x18_Female" H 5400 6600 50  0000 C CNN
-F 2 "Connector_PinSocket_2.54mm:PinSocket_1x18_P2.54mm_Vertical" H 5400 7600 50  0001 C CNN
-F 3 "~" H 5400 7600 50  0001 C CNN
-	1    5400 7600
-	-1   0    0    -1
-$EndComp
-$Comp
-L Connector:Conn_01x18_Male J1
-U 1 1 620F68D3
-P 4850 7600
-F 0 "J1" H 5000 8700 50  0000 R CNN
-F 1 "Conn_01x18_Male" H 5250 8600 50  0000 R CNN
-F 2 "Connector_PinHeader_2.54mm:PinHeader_1x18_P2.54mm_Vertical" H 4850 7600 50  0001 C CNN
-F 3 "~" H 4850 7600 50  0001 C CNN
-	1    4850 7600
-	-1   0    0    -1
 $EndComp
 Wire Wire Line
@@
 	1    15600 9150
 	-1   0    0    -1
-$EndComp
-$Comp
-L Connector:Conn_01x18_Female J7
-U 1 1 62619869
-P 12900 7600
-F 0 "J7" H 12800 8600 50  0000 C CNN
-F 1 "Conn_01x18_Female" H 12900 6600 50  0000 C CNN
-F 2 "Connector_PinSocket_2.54mm:PinSocket_1x18_P2.54mm_Vertical" H 12900 7600 50  0001 C CNN
-F 3 "~" H 12900 7600 50  0001 C CNN
-	1    12900 7600
-	1    0    0    -1
-$EndComp
-$Comp
-L Connector:Conn_01x18_Male J8
-U 1 1 6261986F
-P 13450 7600
-F 0 "J8" H 13600 8700 50  0000 R CNN
-F 1 "Conn_01x18_Male" H 13850 8600 50  0000 R CNN
-F 2 "Connector_PinHeader_2.54mm:PinHeader_1x18_P2.54mm_Vertical" H 13450 7600 50  0001 C CNN
-F 3 "~" H 13450 7600 50  0001 C CNN
-	1    13450 7600
-	1    0    0    -1
 $EndComp
 Wire Wire Line
@@
 Wire Wire Line
 	9150 4450 9150 4550
+$Comp
+L Connector:Conn_01x04_Male J7
+U 1 1 6355EACB
+P 4850 7800
+F 0 "J7" H 4912 7944 50  0000 L CNN
+F 1 "Conn_01x04_Male" H 5003 7944 50  0000 L CNN
+F 2 "Connector_PinHeader_2.54mm:PinHeader_1x04_P2.54mm_Vertical" H 4850 7800 50  0001 C CNN
+F 3 "~" H 4850 7800 50  0001 C CNN
+	1    4850 7800
+	-1   0    0    1
+$EndComp
+$Comp
+L Connector:Conn_01x04_Female J22
+U 1 1 6355FF0A
+P 5400 7800
+F 0 "J22" V 5246 7948 50  0000 L CNN
+F 1 "Conn_01x04_Female" H 5337 7948 50  0000 L CNN
+F 2 "Connector_PinSocket_2.54mm:PinSocket_1x04_P2.54mm_Vertical" H 5400 7800 50  0001 C CNN
+F 3 "~" H 5400 7800 50  0001 C CNN
+	1    5400 7800
+	-1   0    0    1
+$EndComp
+$Comp
+L Connector:Conn_01x04_Female J20
+U 1 1 6364D01C
+P 5400 7000
+F 0 "J20" H 5246 7148 50  0000 L CNN
+F 1 "Conn_01x04_Female" H 5337 7148 50  0000 L CNN
+F 2 "Connector_PinSocket_2.54mm:PinSocket_1x04_P2.54mm_Vertical" H 5400 7000 50  0001 C CNN
+F 3 "~" H 5400 7000 50  0001 C CNN
+	1    5400 7000
+	-1   0    0    1
+$EndComp
+$Comp
+L Connector:Conn_01x04_Male J1
+U 1 1 6365127E
+P 4850 7000
+F 0 "J1" H 4912 7144 50  0000 L CNN
+F 1 "Conn_01x04_Male" H 5003 7144 50  0000 L CNN
+F 2 "Connector_PinHeader_2.54mm:PinHeader_1x04_P2.54mm_Vertical" H 4850 7000 50  0001 C CNN
+F 3 "~" H 4850 7000 50  0001 C CNN
+	1    4850 7000
+	-1   0    0    1
+$EndComp
+$Comp
+L Connector:Conn_01x04_Male J2
+U 1 1 63651670
+P 4850 7400
+F 0 "J2" H 4912 7544 50  0000 L CNN
+F 1 "Conn_01x04_Male" H 5003 7544 50  0000 L CNN
+F 2 "Connector_PinHeader_2.54mm:PinHeader_1x04_P2.54mm_Vertical" H 4850 7400 50  0001 C CNN
+F 3 "~" H 4850 7400 50  0001 C CNN
+	1    4850 7400
+	-1   0    0    1
+$EndComp
+$Comp
+L Connector:Conn_01x04_Female J21
+U 1 1 63650D67
+P 5400 7400
+F 0 "J21" H 5246 7548 50  0000 L CNN
+F 1 "Conn_01x04_Female" H 5337 7548 50  0000 L CNN
+F 2 "Connector_PinSocket_2.54mm:PinSocket_1x04_P2.54mm_Vertical" H 5400 7400 50  0001 C CNN
+F 3 "~" H 5400 7400 50  0001 C CNN
+	1    5400 7400
+	-1   0    0    1
+$EndComp
+$Comp
+L Connector:Conn_01x04_Male J8
+U 1 1 636A5F98
+P 4850 8200
+F 0 "J8" H 4912 8344 50  0000 L CNN
+F 1 "Conn_01x04_Male" H 5003 8344 50  0000 L CNN
+F 2 "Connector_PinHeader_2.54mm:PinHeader_1x04_P2.54mm_Vertical" H 4850 8200 50  0001 C CNN
+F 3 "~" H 4850 8200 50  0001 C CNN
+	1    4850 8200
+	-1   0    0    1
+$EndComp
+$Comp
+L Connector:Conn_01x04_Female J23
+U 1 1 636A4DFA
+P 5400 8200
+F 0 "J23" H 5246 8348 50  0000 L CNN
+F 1 "Conn_01x04_Female" H 5337 8348 50  0000 L CNN
+F 2 "Connector_PinSocket_2.54mm:PinSocket_1x04_P2.54mm_Vertical" H 5400 8200 50  0001 C CNN
+F 3 "~" H 5400 8200 50  0001 C CNN
+	1    5400 8200
+	-1   0    0    1
+$EndComp
+$Comp
+L Connector:Conn_01x04_Male J26
+U 1 1 636DA3DA
+P 12900 7800
+F 0 "J26" H 12962 7944 50  0000 L CNN
+F 1 "Conn_01x04_Male" H 13053 7944 50  0000 L CNN
+F 2 "Connector_PinHeader_2.54mm:PinHeader_1x04_P2.54mm_Vertical" H 12900 7800 50  0001 C CNN
+F 3 "~" H 12900 7800 50  0001 C CNN
+	1    12900 7800
+	-1   0    0    1
+$EndComp
+$Comp
+L Connector:Conn_01x04_Female J30
+U 1 1 636DA3E0
+P 13450 7800
+F 0 "J30" V 13296 7948 50  0000 L CNN
+F 1 "Conn_01x04_Female" H 13387 7948 50  0000 L CNN
+F 2 "Connector_PinSocket_2.54mm:PinSocket_1x04_P2.54mm_Vertical" H 13450 7800 50  0001 C CNN
+F 3 "~" H 13450 7800 50  0001 C CNN
+	1    13450 7800
+	-1   0    0    1
+$EndComp
+$Comp
+L Connector:Conn_01x04_Female J28
+U 1 1 636DA3E6
+P 13450 7000
+F 0 "J28" H 13296 7148 50  0000 L CNN
+F 1 "Conn_01x04_Female" H 13387 7148 50  0000 L CNN
+F 2 "Connector_PinSocket_2.54mm:PinSocket_1x04_P2.54mm_Vertical" H 13450 7000 50  0001 C CNN
+F 3 "~" H 13450 7000 50  0001 C CNN
+	1    13450 7000
+	-1   0    0    1
+$EndComp
+$Comp
+L Connector:Conn_01x04_Male J24
+U 1 1 636DA3EC
+P 12900 7000
+F 0 "J24" H 12962 7144 50  0000 L CNN
+F 1 "Conn_01x04_Male" H 13053 7144 50  0000 L CNN
+F 2 "Connector_PinHeader_2.54mm:PinHeader_1x04_P2.54mm_Vertical" H 12900 7000 50  0001 C CNN
+F 3 "~" H 12900 7000 50  0001 C CNN
+	1    12900 7000
+	-1   0    0    1
+$EndComp
+$Comp
+L Connector:Conn_01x04_Male J25
+U 1 1 636DA3F2
+P 12900 7400
+F 0 "J25" H 12962 7544 50  0000 L CNN
+F 1 "Conn_01x04_Male" H 13053 7544 50  0000 L CNN
+F 2 "Connector_PinHeader_2.54mm:PinHeader_1x04_P2.54mm_Vertical" H 12900 7400 50  0001 C CNN
+F 3 "~" H 12900 7400 50  0001 C CNN
+	1    12900 7400
+	-1   0    0    1
+$EndComp
+$Comp
+L Connector:Conn_01x04_Female J29
+U 1 1 636DA3F8
+P 13450 7400
+F 0 "J29" H 13296 7548 50  0000 L CNN
+F 1 "Conn_01x04_Female" H 13387 7548 50  0000 L CNN
+F 2 "Connector_PinSocket_2.54mm:PinSocket_1x04_P2.54mm_Vertical" H 13450 7400 50  0001 C CNN
+F 3 "~" H 13450 7400 50  0001 C CNN
+	1    13450 7400
+	-1   0    0    1
+$EndComp
+$Comp
+L Connector:Conn_01x04_Male J27
+U 1 1 636DA3FE
+P 12900 8200
+F 0 "J27" H 12962 8344 50  0000 L CNN
+F 1 "Conn_01x04_Male" H 13053 8344 50  0000 L CNN
+F 2 "Connector_PinHeader_2.54mm:PinHeader_1x04_P2.54mm_Vertical" H 12900 8200 50  0001 C CNN
+F 3 "~" H 12900 8200 50  0001 C CNN
+	1    12900 8200
+	-1   0    0    1
+$EndComp
+$Comp
+L Connector:Conn_01x04_Female J31
+U 1 1 636DA404
+P 13450 8200
+F 0 "J31" H 13296 8348 50  0000 L CNN
+F 1 "Conn_01x04_Female" H 13387 8348 50  0000 L CNN
+F 2 "Connector_PinSocket_2.54mm:PinSocket_1x04_P2.54mm_Vertical" H 13450 8200 50  0001 C CNN
+F 3 "~" H 13450 8200 50  0001 C CNN
+	1    13450 8200
+	-1   0    0    1
+$EndComp
 $EndSCHEMATC

Commit message: End of the day resuls
Connections:
- net at MX1.1 (COL): now also J1.4 (Pin_4), MX2.1 (COL), MX3.1 (COL)
- net at MX4.1 (COL): now also J1.3 (Pin_3), MX5.1 (COL), MX6.1 (COL)
- net at MX7.1 (COL): now also J1.2 (Pin_2), MX8.1 (COL), MX9.1 (COL)
- net at MX11.1 (COL): now also J1.1 (Pin_1), MX12.1 (COL), MX13.1 (COL)
- net at MX42.1 (COL): now also J28.4 (Pin_4), MX43.1 (COL), MX44.1 (COL)
- net at MX39.1 (COL): now also J28.3 (Pin_3), MX40.1 (COL), MX41.1 (COL)
Changed lines of the file:
@@
 $EndComp
 Wire Wire Line
-	1450 6350 1450 8300
-Wire Wire Line
-	2150 6400 2150 8300
-Wire Wire Line
-	16850 6350 16850 8300
-Wire Wire Line
-	16150 6400 16150 8300
+	1450 6350 1450 6700
+Wire Wire Line
+	2150 6400 2150 6700
+Wire Wire Line
+	16850 6350 16850 6700
+Wire Wire Line
+	16150 6400 16150 6700
 Wire Wire Line
 	8950 6250 8950 8750
@@
 	3350 9400 6550 9400
 Wire Wire Line
-	2850 8300 2850 6450
-Wire Wire Line
-	3550 6500 3550 8300
+	2850 8300 2850 7500
+Wire Wire Line
+	3550 6500 3550 6700
 Wire Wire Line
 	3550 9100 6300 9100
@@
 	-1   0    0    1
 $EndComp
+Connection ~ 1450 6700
+Wire Wire Line
+	1450 6700 1450 7500
+Connection ~ 1450 7500
+Wire Wire Line
+	1450 7500 1450 8300
+Connection ~ 1450 8300
+Connection ~ 2150 8300
+Connection ~ 2150 7500
+Wire Wire Line
+	2150 7500 2150 8300
+Connection ~ 2150 6700
+Wire Wire Line
+	2150 6700 2150 7500
+Connection ~ 2850 6700
+Wire Wire Line
+	2850 6700 2850 6450
+Connection ~ 3550 6700
+Wire Wire Line
+	3550 6700 3550 7500
+Connection ~ 3550 7500
+Wire Wire Line
+	3550 7500 3550 8300
+Connection ~ 2850 7500
+Wire Wire Line
+	2850 7500 2850 6700
+Connection ~ 2850 8300
+Connection ~ 3550 8300
+Connection ~ 16150 6700
+Wire Wire Line
+	16150 6700 16150 7500
+Connection ~ 16150 7500
+Wire Wire Line
+	16150 7500 16150 8300
+Connection ~ 16850 7500
+Wire Wire Line
+	16850 7500 16850 8300
+Connection ~ 16850 6700
+Wire Wire Line
+	16850 6700 16850 7500
+Connection ~ 16850 8300
+Connection ~ 16150 8300
+Connection ~ 15450 8300
+Connection ~ 14750 8300
 $EndSCHEMATC

Commit message: End of the day resuls
Connections:
- net COL4: now also MX15.1 (COL), MX16.1 (COL), MX17.1 (COL)
- net COL5: now also MX19.1 (COL), MX20.1 (COL), MX21.1 (COL)
- net COL6: now also MX23.1 (COL), MX24.1 (COL), MX25.1 (COL)
- net COL7: now also MX27.1 (COL), MX28.1 (COL), MX29.1 (COL)
Changed lines of the file:
@@
 	16150 6400 16150 6700
 Wire Wire Line
-	8950 6250 8950 8750
-Wire Wire Line
-	8250 6250 8250 9850
-Wire Wire Line
-	10300 6250 10300 9900
-Wire Wire Line
-	9600 6250 9600 8750
+	8950 6250 8950 6550
+Wire Wire Line
+	8250 6250 8250 6550
+Wire Wire Line
+	10300 6250 10300 6550
+Wire Wire Line
+	9600 6250 9600 6550
 Text GLabel 8250 6250 1    50   Input ~ 0
 COL4
@@
 Wire Wire Line
 	1450 7500 1450 8300
-Connection ~ 1450 8300
-Connection ~ 2150 8300
 Connection ~ 2150 7500
 Wire Wire Line
@@
 Wire Wire Line
 	2850 7500 2850 6700
-Connection ~ 2850 8300
-Connection ~ 3550 8300
 Connection ~ 16150 6700
 Wire Wire Line
@@
 Wire Wire Line
 	16850 6700 16850 7500
-Connection ~ 16850 8300
-Connection ~ 16150 8300
-Connection ~ 15450 8300
-Connection ~ 14750 8300
+Connection ~ 8250 6550
+Wire Wire Line
+	8250 6550 8250 7350
+Connection ~ 8250 7350
+Wire Wire Line
+	8250 7350 8250 8150
+Connection ~ 8250 8150
+Wire Wire Line
+	8250 8150 8250 9850
+Connection ~ 8950 8150
+Wire Wire Line
+	8950 8150 8950 8750
+Connection ~ 9600 8150
+Wire Wire Line
+	9600 8150 9600 8750
+Connection ~ 10300 8150
+Wire Wire Line
+	10300 8150 10300 9900
+Connection ~ 10300 7350
+Wire Wire Line
+	10300 7350 10300 8150
+Connection ~ 9600 7350
+Wire Wire Line
+	9600 7350 9600 8150
+Connection ~ 8950 7350
+Wire Wire Line
+	8950 7350 8950 8150
+Connection ~ 8950 6550
+Wire Wire Line
+	8950 6550 8950 7350
+Connection ~ 9600 6550
+Wire Wire Line
+	9600 6550 9600 7350
+Connection ~ 10300 6550
+Wire Wire Line
+	10300 6550 10300 7350
 $EndSCHEMATC

Commit message: Somewhat completed the development
Parts:
- J19: footprint 525591233 -> 52559-1233:525591233
Connections:
- net SCL: no longer J17.3 (Pin_3), J19.9
- net SDA: no longer J17.2 (Pin_2), J19.10
- new net SCL-TOP: J17.3 (Pin_3), J19.9
- new net SDA-TOP: J17.2 (Pin_2), J19.10
Changed lines of the file:
@@
 F 0 "J19" H 11400 3615 50  0000 C CNN
 F 1 "52559-1233" H 11400 3524 50  0000 C CNN
-F 2 "525591233" H 11750 3450 50  0001 L CNN
+F 2 "52559-1233:525591233" H 11750 3450 50  0001 L CNN
 F 3 "" H 11750 3350 50  0001 L CNN
 F 4 "FFC & FPC Connectors 0.5 FPC ZIF 12Ckt Sn-Ag-Bi" H 11750 3250 50  0001 L CNN "Description"
@@
 $EndComp
 Text GLabel 10900 3850 0    50   Input ~ 0
-SCL
+SCL-TOP
 Text GLabel 11900 3850 2    50   Input ~ 0
-SDA
+SDA-TOP
 $Comp
 L power:VCC #PWR0101
@@
 SCL
 Text GLabel 9450 3900 1    50   Input ~ 0
-SCL
+SCL-TOP
 Text GLabel 9550 3900 1    50   Input ~ 0
-SDA
+SDA-TOP
 $Comp
 L power:GND #PWR0103
